Commit message: rosbag data

File: src/amr_description/urdf/amr.urdf.xacro (robot description, xacro)
@@ -358,5 +358,6 @@
     <parent link="base_link"/>
     <child link="laser_link"/>
-    <origin xyz="0 0 0.29" rpy="0 0 0"/>   <!--  modify height of rp lidar here -->
+    <origin xyz="0 0 0.24" rpy="0 0 0"/>   <!--  modify height of rp lidar here -->
+    <!--  top shelf 0.29 -->
   </joint>
   <link name="laser_link">
