Commit message: edit publish rate to 100 Hz except motion genertor 5 Hz and create launch file for testing KC

File: src/amr_description/urdf/amr.urdf_blue.xacro (robot description, xacro)
@@ -17,5 +17,5 @@
     <inertial>
       <origin xyz="0 0 0.0" rpy="0 0 0"/>
-      <mass value="20"/>
+      <mass value="40"/>
       <inertia ixx="0.33" ixy="0" ixz="0" iyy="0.54" iyz="0" izz="0.77"/>
     </inertial>

File: src/amr_description/urdf/amr.urdf_red.xacro (robot description, xacro)
@@ -17,5 +17,5 @@
     <inertial>
       <origin xyz="0 0 0.0" rpy="0 0 0"/>
-      <mass value="20"/>
+      <mass value="40"/>
       <inertia ixx="0.33" ixy="0" ixz="0" iyy="0.54" iyz="0" izz="0.77"/>
     </inertial>
