Commit message: edit urdf roll back to planar move

File: src/amr_description/urdf/amr.gazebo_red.xacro (robot description, xacro)
@@ -5,4 +5,7 @@
   <gazebo reference="base_link">
     <material>Gazebo/Red</material>
+    <mu1>2.0</mu1>
+    <mu2>2.0</mu2>
+    <fdir1>1 0 0</fdir1>
   </gazebo>
   <gazebo reference="bumper_link">

File: src/amr_description/urdf/amr.urdf_blue.xacro (robot description, xacro)
@@ -349,4 +349,5 @@
   </joint>
   <link name="imu_link"/>
+<!--
   <joint name="scan_joint" type="fixed">
     <parent link="laser_link"/>
@@ -358,5 +359,6 @@
     <parent link="base_link"/>
     <child link="laser_link"/>
-    <origin xyz="0 0 0.29" rpy="0 0 0"/>   <!--  modify height of rp lidar here -->
+    <origin xyz="0 0 0.29" rpy="0 0 0"/>   -->  <!--  modify height of rp lidar here -->
+  <!--
   </joint>
   <link name="laser_link">
@@ -379,4 +381,5 @@
     </inertial>
   </link>
+-->
   <!--
   <joint name="camera_joint" type="fixed">

File: src/amr_description/urdf/amr.urdf_red.xacro (robot description, xacro)
@@ -349,4 +349,5 @@
   </joint>
   <link name="imu_link"/>
+<!--
   <joint name="scan_joint" type="fixed">
     <parent link="laser_link"/>
@@ -358,6 +359,6 @@
     <parent link="base_link"/>
     <child link="laser_link"/>
-    <origin xyz="0 0 0.24" rpy="0 0 0"/>   <!--  modify height of rp lidar here -->
-    <!--  top shelf 0.29 -->
+    <origin xyz="0 0 0.29" rpy="0 0 0"/>   -->  <!--  modify height of rp lidar here -->
+  <!--
   </joint>
   <link name="laser_link">
@@ -380,4 +381,5 @@
     </inertial>
   </link>
+-->
   <!--
   <joint name="camera_joint" type="fixed">
