Commit message: latest update force based controller

File: src/amr_description/urdf/amr.gazebo_blue.xacro (robot description, xacro)
@@ -75,5 +75,5 @@
       <jointName>wheel_fl_joint, wheel_fr_joint, wheel_rl_joint, wheel_rr_joint</jointName>
       <robotNameSpace>/</robotNameSpace>
-      <updateRate>100</updateRate>
+      <updateRate>100.0</updateRate>
     </plugin>
   </gazebo>
@@ -103,11 +103,11 @@
       <commandTopic>cmd_vel</commandTopic>
       <odometryTopic>odom</odometryTopic>
-      <odometryFrame>odom</odometryFrame>
+      <odometryFrame>map</odometryFrame>
       <odometryRate>100.0</odometryRate>
       <robotBaseFrame>base_link</robotBaseFrame>
-      <publish_odom_tf>true </publish_odom_tf>
-      <yaw_velocity_p_gain>150</yaw_velocity_p_gain>
+      <publishOdometryTf>true </publishOdometryTf>
+      <yaw_velocity_p_gain>100</yaw_velocity_p_gain>
       <x_velocity_p_gain>15</x_velocity_p_gain>
-      <y_velocity_p_gain>15</y_velocity_p_gain>
+      <y_velocity_p_gain>500</y_velocity_p_gain>
     </plugin>
   </gazebo>

File: src/amr_description/urdf/amr.gazebo_red.xacro (robot description, xacro)
@@ -107,5 +107,5 @@
       <robotBaseFrame>base_link</robotBaseFrame>
       <publish_odom_tf>true </publish_odom_tf>
-      <yaw_velocity_p_gain>150</yaw_velocity_p_gain>
+      <yaw_velocity_p_gain>100</yaw_velocity_p_gain>
       <x_velocity_p_gain>15</x_velocity_p_gain>
       <y_velocity_p_gain>15</y_velocity_p_gain>

File: src/amr_description/urdf/amr.urdf_blue.xacro (robot description, xacro)
@@ -17,5 +17,5 @@
     <inertial>
       <origin xyz="0 0 0.0" rpy="0 0 0"/>
-      <mass value="40"/>
+      <mass value="20"/>
       <inertia ixx="0.33" ixy="0" ixz="0" iyy="0.54" iyz="0" izz="0.77"/>
     </inertial>
@@ -358,6 +358,5 @@
     <parent link="base_link"/>
     <child link="laser_link"/>
-    <origin xyz="0 0 0.24" rpy="0 0 0"/>   <!--  modify height of rp lidar here -->
-    <!--  top shelf 0.29 -->
+    <origin xyz="0 0 0.29" rpy="0 0 0"/>   <!--  modify height of rp lidar here -->
   </joint>
   <link name="laser_link">

Commit message: edit with ridgeback robot

File: src/amr_description/urdf/amr.gazebo_blue.xacro (robot description, xacro)
@@ -103,13 +103,30 @@
       <commandTopic>cmd_vel</commandTopic>
       <odometryTopic>odom</odometryTopic>
-      <odometryFrame>map</odometryFrame>
+      <odometryFrame>odom</odometryFrame>
       <odometryRate>100.0</odometryRate>
       <robotBaseFrame>base_link</robotBaseFrame>
-      <publishOdometryTf>true </publishOdometryTf>
+      <publishOdometryTf>true</publishOdometryTf>
       <yaw_velocity_p_gain>100</yaw_velocity_p_gain>
-      <x_velocity_p_gain>15</x_velocity_p_gain>
-      <y_velocity_p_gain>500</y_velocity_p_gain>
-    </plugin>
-  </gazebo>
+      <x_velocity_p_gain>150</x_velocity_p_gain>
+      <y_velocity_p_gain>1000</y_velocity_p_gain>
+      <cmdVelTimeOut>0.25</cmdVelTimeOut>
+    </plugin>
+  </gazebo>
+  <!--
+   <gazebo>
+     <plugin name="ridgeback_ros_force_based_move" filename="libridgeback_ros_force_based_move.so">
+      <commandTopic>cmd_vel</commandTopic>
+      <odometryTopic>odom</odometryTopic>
+      <odometryFrame>odom</odometryFrame>
+      <odometryRate>100</odometryRate>
+      <robotBaseFrame>base_link</robotBaseFrame>
+      <cmdVelTimeOut>0.25</cmdVelTimeOut>
+      <publishOdometryTf>false</publishOdometryTf>
+      <yaw_velocity_p_gain>300.0</yaw_velocity_p_gain>
+      <x_velocity_p_gain>200</x_velocity_p_gain>
+      <y_velocity_p_gain>5000</y_velocity_p_gain>
+    </plugin>
+    </gazebo>
+    -->
    <!--
    <gazebo>

File: src/amr_description/urdf/amr.gazebo_red.xacro (robot description, xacro)
@@ -99,5 +99,5 @@
   </gazebo>
   -->
-<gazebo>
+    <gazebo>
    <plugin name="ros_force_based_controller" filename="libgazebo_ros_force_based_move.so">
       <commandTopic>cmd_vel</commandTopic>
@@ -106,8 +106,9 @@
       <odometryRate>100.0</odometryRate>
       <robotBaseFrame>base_link</robotBaseFrame>
-      <publish_odom_tf>true </publish_odom_tf>
+      <publishOdometryTf>true </publishOdometryTf>
       <yaw_velocity_p_gain>100</yaw_velocity_p_gain>
-      <x_velocity_p_gain>15</x_velocity_p_gain>
-      <y_velocity_p_gain>15</y_velocity_p_gain>
+      <x_velocity_p_gain>150</x_velocity_p_gain>
+      <y_velocity_p_gain>1000</y_velocity_p_gain>
+      <cmdVelTimeOut>0.25</cmdVelTimeOut>
     </plugin>
   </gazebo>

File: src/amr_description/urdf/amr.urdf_blue.xacro (robot description, xacro)
@@ -17,5 +17,5 @@
     <inertial>
       <origin xyz="0 0 0.0" rpy="0 0 0"/>
-      <mass value="20"/>
+      <mass value="40"/>
       <inertia ixx="0.33" ixy="0" ixz="0" iyy="0.54" iyz="0" izz="0.77"/>
     </inertial>

Commit message: edit urdf to remove top plate

File: src/amr_description/urdf/amr.gazebo_blue.xacro (robot description, xacro)
@@ -5,6 +5,6 @@
   <gazebo reference="base_link">
     <material>Gazebo/Blue</material>
-    <mu1>2.0</mu1>
-    <mu2>2.0</mu2>
+    <mu1>20.0</mu1>
+    <mu2>20.0</mu2>
     <fdir1>1 0 0</fdir1>
   </gazebo>
@@ -12,8 +12,8 @@
     <material>Gazebo/Grey</material>
   </gazebo>
+    <!--
   <gazebo reference="plate_link1">
     <material>Gazebo/Grey</material>
   </gazebo>
-  <!--
   <gazebo reference="plate_link2">
     <material>Gazebo/Grey</material>

File: src/amr_description/urdf/amr.gazebo_force_based.xacro (robot description, xacro)
@@ -4,5 +4,5 @@
   <xacro:arg name="imu_visual"   default="false"/>
   <gazebo reference="base_link">
-    <material>Gazebo/Red</material>
+    <material>Gazebo/Yellow</material>
     <mu1>20.0</mu1>
     <mu2>20.0</mu2>
@@ -77,30 +77,11 @@
       <alwaysOn>true</alwaysOn>
       <jointName>wheel_fl_joint, wheel_fr_joint, wheel_rl_joint, wheel_rr_joint</jointName>
-      <robotNameSpace>/</robotNameSpace>
-      <updateRate>100</updateRate>
-    </plugin>
-  </gazebo>
- <!--
-  <gazebo>
-    <plugin name="skid_steer_drive_controller" filename="libgazebo_ros_skid_steer_drive.so">
-      <alwaysOn>true</alwaysOn>
-      <updateRate>50.0</updateRate>
-      <robotNamespace>/</robotNamespace>
-      <leftFrontJoint>wheel_fl_joint</leftFrontJoint>
-      <rightFrontJoint>wheel_fr_joint</rightFrontJoint>
-      <leftRearJoint>wheel_rl_joint</leftRearJoint>
-      <rightRearJoint>wheel_rr_joint</rightRearJoint>
-      <wheelSeparation>0.334</wheelSeparation>
-      <wheelDiameter>0.144</wheelDiameter>
-      <robotBaseFrame>base_link</robotBaseFrame>
-      <torque>20</torque>
-      <commandTopic>cmd_vel</commandTopic>
-      <odometryTopic>odom</odometryTopic>
-      <odometryFrame>odom</odometryFrame>
-      <broadcastTF>true</broadcastTF>
-    </plugin>
-  </gazebo>
-  -->
-  <!--
+    <!-- Name space tag may be removed
+      <robotNamespace>$(arg name_space)</robotNamespace>
+      -->
+      <updateRate>100.0</updateRate>
+    </plugin>
+  </gazebo>
+   <!--
     <gazebo>
    <plugin name="ros_force_based_controller" filename="libgazebo_ros_force_based_move.so">
@@ -110,5 +91,5 @@
       <odometryRate>100.0</odometryRate>
       <robotBaseFrame>base_link</robotBaseFrame>
-      <publishOdometryTf>true </publishOdometryTf>
+      <publishOdometryTf>true</publishOdometryTf>
       <yaw_velocity_p_gain>100</yaw_velocity_p_gain>
       <x_velocity_p_gain>150</x_velocity_p_gain>
@@ -117,5 +98,15 @@
     </plugin>
   </gazebo>
- <gazebo>
+ -->
+   <gazebo>
+    <plugin name="gazebo_ros_control" filename="libgazebo_ros_control.so">
+        <!-- Name space tag may be removed
+      <robotNamespace>$(arg name_space)</robotNamespace>
+      -->
+      <robotParam>robot_description</robotParam>
+       <legacyModeNS>true</legacyModeNS>
+    </plugin>
+</gazebo>
+   <gazebo>
      <plugin name="ridgeback_ros_force_based_move" filename="libridgeback_ros_force_based_move.so">
       <commandTopic>cmd_vel</commandTopic>
@@ -131,42 +122,21 @@
     </plugin>
     </gazebo>
--->
-   <gazebo>
-    <plugin filename="libgazebo_ros_planar_move.so" name="amr_planar_controller">
-      <commandTopic>cmd_vel</commandTopic>
-      <odometryTopic>odom</odometryTopic>
-      <odometryFrame>odom</odometryFrame>
-      <odometryRate>100</odometryRate>
-      <robotBaseFrame>base_link</robotBaseFrame>
-    </plugin>
-  </gazebo>
-  <gazebo>
-    <plugin name="imu_plugin" filename="libgazebo_ros_imu.so">
-      <alwaysOn>true</alwaysOn>
-      <bodyName>imu_link</bodyName>
-      <frameName>imu_link</frameName>
-      <topicName>imu</topicName>
-      <serviceName>imu_service</serviceName>
-      <gaussianNoise>0.0</gaussianNoise>
-      <updateRate>100</updateRate>
-      <imu>
-        <noise>
-          <type>gaussian</type>
-          <rate>
-            <mean>0.0</mean>
-            <stddev>2e-4</stddev>
-            <bias_mean>0.0000075</bias_mean>
-            <bias_stddev>0.0000008</bias_stddev>
-          </rate>
-          <accel>
-            <mean>0.0</mean>
-            <stddev>1.7e-2</stddev>
-            <bias_mean>0.1</bias_mean>
-            <bias_stddev>0.001</bias_stddev>
-          </accel>
-        </noise>
-      </imu>
-    </plugin>
-  </gazebo>
+     <gazebo>
+      <plugin name="imu_controller" filename="libhector_gazebo_ros_imu.so">
+        <!--<robotNamespace>$(arg name_space)</robotNamespace>
+        <frameId>$(arg name_space)/base_link</frameId>
+        -->
+        <robotParam>robot_description</robotParam>
+        <updateRate>100.0</updateRate>
+        <bodyName>base_link</bodyName>
+        <topicName>imu/data</topicName>
+        <accelDrift>0.005 0.005 0.005</accelDrift>
+        <accelGaussianNoise>0.005 0.005 0.005</accelGaussianNoise>
+        <rateDrift>0.005 0.005 0.005 </rateDrift>
+        <rateGaussianNoise>0.005 0.005 0.005 </rateGaussianNoise>
+        <headingDrift>0.005</headingDrift>
+        <headingGaussianNoise>0.005</headingGaussianNoise>
+      </plugin>
+    </gazebo>
 <!--
   <gazebo reference="base_scan">

File: src/amr_description/urdf/amr.gazebo_green.xacro (robot description, xacro)
@@ -5,6 +5,6 @@
   <gazebo reference="base_link">
     <material>Gazebo/Green</material>
-    <mu1>2.0</mu1>
-    <mu2>2.0</mu2>
+    <mu1>20.0</mu1>
+    <mu2>20.0</mu2>
     <fdir1>1 0 0</fdir1>
   </gazebo>
@@ -12,8 +12,8 @@
     <material>Gazebo/Grey</material>
   </gazebo>
+   <!--
   <gazebo reference="plate_link1">
     <material>Gazebo/Grey</material>
   </gazebo>
-  <!--
   <gazebo reference="plate_link2">
     <material>Gazebo/Grey</material>

File: src/amr_description/urdf/amr.urdf_blue.xacro (robot description, xacro)
@@ -45,4 +45,5 @@
     </inertial>
   </link>
+  <!--
   <joint name="plate_joint1" type="fixed">
     <parent link="base_link"/>
@@ -105,5 +106,4 @@
     </inertial>
   </link>
-  <!--
    <joint name="plate_joint2" type="fixed">
     <parent link="base_link"/>

File: src/amr_description/urdf/amr.urdf_force_based.xacro (robot description, xacro)
@@ -1,5 +1,5 @@
 <?xml version="1.0" ?>
 <robot name="amr" xmlns:xacro="http://ros.org/wiki/xacro">
-  <xacro:include filename="$(find amr_description)/urdf/amr.gazebo_green.xacro"/>
+  <xacro:include filename="$(find amr_description)/urdf/amr.gazebo_force_based.xacro"/>
   <link name="base_link">
     <visual>
@@ -45,5 +45,4 @@
     </inertial>
   </link>
-  <!--
   <joint name="plate_joint1" type="fixed">
     <parent link="base_link"/>
@@ -106,4 +105,5 @@
     </inertial>
   </link>
+  <!--
    <joint name="plate_joint2" type="fixed">
     <parent link="base_link"/>
@@ -358,5 +358,5 @@
     <parent link="base_link"/>
     <child link="laser_link"/>
-    <origin xyz="0 0 0.65" rpy="0 0 0"/>     <!--  modify height of rp lidar here -->
+    <origin xyz="0 0 0.29" rpy="0 0 0"/>     <!--  modify height of rp lidar here -->
   </joint>
   <link name="laser_link">

File: src/amr_description/urdf/amr.urdf_red.xacro (robot description, xacro)
@@ -45,4 +45,5 @@
     </inertial>
   </link>
+   <!--
   <joint name="plate_joint1" type="fixed">
     <parent link="base_link"/>
@@ -105,5 +106,4 @@
     </inertial>
   </link>
-  <!--
    <joint name="plate_joint2" type="fixed">
     <parent link="base_link"/>

File: src/amr_description/urdf/load.urdf (robot description, URDF)
Before this commit: robot simple_box, 1 links, 0 joints
Links:
- link my_box: geometry collision box size=2 2 0.1; visual box size=2 2 0.1
