Commit message: edit vl force node paramater from vl to vl_robot

File: src/amr_description/urdf/load.urdf (robot description, URDF)
Before this commit: robot simple_box, 1 links, 0 joints
Links:
- link my_box: mass 1.0 -> 100.0; geometry collision box size=1.45 1.45 0.1; visual box size=1.45 1.45 0.1

Commit message: latest edit

File: src/amr_description/urdf/load.urdf (robot description, URDF)
Before this commit: robot simple_box, 1 links, 0 joints
Links:
- link my_box: mass 100.0 -> 200.0
