Commit message: update

File: src/amr_description/urdf/load_big.urdf (robot description, URDF)
Before this commit: robot simple_box, 1 links, 0 joints
Links:
- link my_box: mass 300.0 -> 500.0; geometry collision box size=5 5 0.2; visual box size=5 5 0.2

Commit message: update experiment

File: src/amr_description/urdf/load_big.urdf (robot description, URDF)
Before this commit: robot simple_box, 1 links, 0 joints
Links:
- link my_box: mass 500.0 -> 550.0
